File: KiCad/folour/folour.kicad_pcb (KiCad board)
At the start: 2 copper layers, 30 parts, among them J1 Conn_01x02, J2 Conn_01x03, J3 Conn_01x03, J4 Conn_01x03, J5 Conn_01x03, J6 Conn_01x02, SW1 SW_Push, SW2 SW_Push, SW3 SW_Push, SW4 SW_Push, U1 74HC165, U2 74AHC595, U3 74AHC595

Commit message: edited footprint
Parts:
- added R13: 10k, Resistor_THT:R_Axial_DIN0207_L6.3mm_D2.5mm_P10.16mm_Horizontal, F.Cu at (101.1, 100.8)
- added R14: 10k, Resistor_THT:R_Axial_DIN0207_L6.3mm_D2.5mm_P10.16mm_Horizontal, F.Cu at (101.1, 104.8)
- added R15: 10k, Resistor_THT:R_Axial_DIN0207_L6.3mm_D2.5mm_P10.16mm_Horizontal, F.Cu at (101.1, 108.9)
- added R16: 10k, Resistor_THT:R_Axial_DIN0207_L6.3mm_D2.5mm_P10.16mm_Horizontal, F.Cu at (101.1, 112.9)
- D1, D2, D3, D4: value LED_RAGB -> LED_RKGB
- R1, R10, R11, R12, R2, R3, R4, R5, R6, R7, R8, R9: footprint Resistor_THT:R_Axial_DIN0207_L6.3mm_D2.5mm_P7.62mm_Horizontal -> Resistor_THT:R_Axial_DIN0207_L6.3mm_D2.5mm_P10.16mm_Horizontal
- SW1, SW2, SW3, SW4: footprint Button_Switch_THT:SW_PUSH_6mm -> Button_Switch_THT:SW_PUSH-12mm
- U2, U3: value 74AHC595 -> 74HC595
- moved SW4 24.8 mm to (115.0, 102.1)
- moved SW3 17.8 mm to (115.0, 86.5)
- moved D5 13.4 mm to (152.5, 74.8)
- moved SW2 10.8 mm to (115.0, 71.0)
- moved J1 9.13 mm to (146.6, 73.6)
- moved J6 9.13 mm to (146.6, 77.6)
- moved D1 7.65 mm to (131.2, 75.8)
- moved D2 7.65 mm to (131.2, 83.4)
- moved D3 7.65 mm to (131.2, 90.9)
- moved D4 7.65 mm to (131.2, 98.5)
- moved J2 7.65 mm to (140.8, 73.6)
- moved J3 7.65 mm to (140.8, 78.6)
- moved J4 7.65 mm to (140.8, 83.7)
- moved J5 7.65 mm to (140.8, 88.7)
- moved U1 7.65 mm to (131.2, 52.2)
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